File: charger-schdoc.sch (KiCad schematic (older format))
At the start: 57 parts, among them P1 Header 8, P2 5V_OUTPUT, U1 MCP73871-3CAI/ML, U3 TPS61090RSAR

Commit message: remove usb
Parts:
- removed Micro~USB: USB3075-30-A, symbol charger-schdoc-rescue:USB3075-30-A-
Changed lines of the file:
@@
 L power:VBUS VBUS_6
 U 1 1 60ED9948
-P 1450 1950
-F 0 "VBUS_6" H 1450 1950 20  0000 C CNN
-F 1 "VBUS" H 1450 1880 30  0000 C CNN
-F 2 "" H 1450 1950 70  0000 C CNN
-F 3 "" H 1450 1950 70  0000 C CNN
-	1    1450 1950
+P 1350 1800
+F 0 "VBUS_6" H 1350 1800 20  0000 C CNN
+F 1 "VBUS" H 1350 1730 30  0000 C CNN
+F 2 "" H 1350 1800 70  0000 C CNN
+F 3 "" H 1350 1800 70  0000 C CNN
+	1    1350 1800
 	1    0    0    -1
 $EndComp
@@
 L power:GND GND_7
 U 1 1 60ED9947
-P 1150 3450
-F 0 "GND_7" H 1150 3590 20  0000 C CNN
-F 1 "GND" H 1150 3560 30  0000 C CNN
-F 2 "" H 1150 3450 70  0000 C CNN
-F 3 "" H 1150 3450 70  0000 C CNN
-	1    1150 3450
+P 1050 3300
+F 0 "GND_7" H 1050 3440 20  0000 C CNN
+F 1 "GND" H 1050 3410 30  0000 C CNN
+F 2 "" H 1050 3300 70  0000 C CNN
+F 3 "" H 1050 3300 70  0000 C CNN
+	1    1050 3300
 	1    0    0    -1
 $EndComp
@@
 	8950 2650 7350 2650
 Wire Wire Line
-	1450 2250 1450 1950
-Wire Wire Line
-	2050 2250 1450 2250
-Wire Wire Line
-	1150 2250 1450 2250
-Wire Wire Line
-	1150 2550 1150 2250
-Wire Wire Line
-	1750 2650 2050 2650
-Wire Wire Line
-	1750 2850 1750 2650
-Wire Wire Line
-	2050 2850 1750 2850
-Wire Wire Line
-	1750 2950 2050 2950
-Wire Wire Line
-	1750 2850 1750 2950
-Wire Wire Line
-	1750 3050 1750 2950
-Wire Wire Line
-	2050 3050 1750 3050
-Wire Wire Line
-	1750 3150 1750 3050
-Wire Wire Line
-	2050 3150 1750 3150
-Wire Wire Line
-	1750 3250 1750 3150
-Wire Wire Line
-	2050 3250 1750 3250
-Wire Wire Line
-	1750 3350 1750 3250
-Wire Wire Line
-	2050 3350 1750 3350
-Wire Wire Line
-	1150 3350 1750 3350
+	1350 2100 1350 1800
+Wire Wire Line
+	1950 2100 1350 2100
+Wire Wire Line
+	1050 2100 1350 2100
+Wire Wire Line
+	1050 2400 1050 2100
+Wire Wire Line
+	1650 2500 1950 2500
+Wire Wire Line
+	1650 2700 1650 2500
+Wire Wire Line
+	1950 2700 1650 2700
+Wire Wire Line
+	1650 2800 1950 2800
+Wire Wire Line
+	1650 2700 1650 2800
+Wire Wire Line
+	1650 2900 1650 2800
+Wire Wire Line
+	1950 2900 1650 2900
+Wire Wire Line
+	1650 3000 1650 2900
+Wire Wire Line
+	1950 3000 1650 3000
+Wire Wire Line
+	1650 3100 1650 3000
+Wire Wire Line
+	1950 3100 1650 3100
+Wire Wire Line
+	1650 3200 1650 3100
+Wire Wire Line
+	1950 3200 1650 3200
+Wire Wire Line
+	1050 3200 1650 3200
 Wire Wire Line
 	1050 5150 2950 5150
@@
 	4950 6650 4950 6350
 Wire Wire Line
-	1150 3350 1150 2850
-Wire Wire Line
-	1150 3450 1150 3350
+	1050 3200 1050 2700
+Wire Wire Line
+	1050 3300 1050 3200
 Text Label 4950 6350 0    60   ~ 0
 Vfb
@@
 Connection ~ 1050 5450
 Connection ~ 1050 5150
-Connection ~ 1150 3350
+Connection ~ 1050 3200
 Connection ~ 1450 5450
-Connection ~ 1450 2250
+Connection ~ 1350 2100
 Connection ~ 1750 7050
 Connection ~ 1750 6450
 Connection ~ 1750 5450
-Connection ~ 1750 3350
-Connection ~ 1750 3250
-Connection ~ 1750 3150
-Connection ~ 1750 3050
-Connection ~ 1750 2950
-Connection ~ 1750 2850
+Connection ~ 1650 3200
+Connection ~ 1650 3100
+Connection ~ 1650 3000
+Connection ~ 1650 2900
+Connection ~ 1650 2800
+Connection ~ 1650 2700
 Connection ~ 2650 5450
 Connection ~ 4550 6250
@@
 $EndComp
 $Comp
-L charger-schdoc-rescue:USB3075-30-A- Micro~USB
-U 1 1 60ED9936
-P 2450 2550
-F 0 "Micro USB" H 2150 2950 60  0000 L BNN
-F 1 "USB3075-30-A" H 2150 1550 60  0000 L BNN
-F 2 "" H 2150 1550 60  0000 C CNN
-F 3 "" H 2150 1550 60  0000 C CNN
-	1    2450 2550
-	1    0    0    -1
-$EndComp
-$Comp
 L charger-schdoc-rescue:TPS61090RSAR- U3
 U 1 1 60ED9935
@@
 L charger-schdoc-rescue:Cap_Pol3- IC
 U 1 1 60ED9926
-P 1250 2650
-F 0 "" H 1250 2650 50  0001 C CNN
-F 1 "" H 1250 2650 50  0001 C CNN
-F 2 "" H 1250 2650 50  0001 C CNN
-F 3 "" H 1250 2650 50  0001 C CNN
-	1    1250 2650
+P 1150 2500
+F 0 "" H 1150 2500 50  0001 C CNN
+F 1 "" H 1150 2500 50  0001 C CNN
+F 2 "" H 1150 2500 50  0001 C CNN
+F 3 "" H 1150 2500 50  0001 C CNN
+	1    1150 2500
 	0    1    1    0
 $EndComp
